Commit message: new double camera

File: urdf/2wv5.urdf (robot description, URDF)
Before this commit: robot 2wv5, 12 links, 11 joints
Links:
- link ball_link_bl: mass 0.204706177307911 -> None; geometry collision sphere radius=0.025; visual sphere radius=0.025
- link ball_link_br: mass 0.204706177307911 -> None; geometry collision sphere radius=0.025; visual sphere radius=0.025
- link ball_link_fl: mass 0.204706177307911 -> None; geometry collision sphere radius=0.025; visual sphere radius=0.025
- link ball_link_fr: mass 0.204706177307911 -> None; geometry collision sphere radius=0.025; visual sphere radius=0.025
- link base_link: mass 62.522 -> None; geometry 
- link chassis_link: geometry collision mesh filename=package://robot_urdf/meshes/2w/chassis_link.STL; visual mesh filename=package://robot_urdf/meshes/2w/chassis_link.STL
- link depth_link_l: mass 62.5218920640007 -> None; geometry 
- link depth_link_r: mass 62.5218920640007 -> None; geometry 
- link left_wheel_holder_link: geometry collision mesh filename=package://robot_urdf/meshes/2w/left_wheel_holder_link.STL; visual mesh filename=package://robot_urdf/meshes/2w/left_wheel_holder_link.STL
- link left_wheel_link: geometry collision mesh filename=package://robot_urdf/meshes/2w/left_wheel_link.STL; visual mesh filename=package://robot_urdf/meshes/2w/left_wheel_link.STL
- link right_wheel_holder_link: geometry collision mesh filename=package://robot_urdf/meshes/2w/right_wheel_holder_link.STL; visual mesh filename=package://robot_urdf/meshes/2w/right_wheel_holder_link.STL
- link right_wheel_link: geometry collision mesh filename=package://robot_urdf/meshes/2w/right_wheel_link.STL; visual mesh filename=package://robot_urdf/meshes/2w/right_wheel_link.STL
Joints:
- joint ball_joint_br: origin xyz=-0.76256 -0.6072 -0.93832 rpy=3.1416 0 3.1416 -> xyz=-0.76256 -0.6072 -0.93832 rpy=0 0 0
- joint depth_joint_l: origin xyz=1.017 0.45 -0.21645 rpy=0 0 -0.2618 -> xyz=1.017 0.45 -0.21645 rpy=0 0.7853982 -0.2618
- joint depth_joint_r: origin xyz=1.017 -0.45 -0.21645 rpy=0 0 0.2618 -> xyz=1.017 -0.45 -0.21645 rpy=0 0.7853982 0.2618
