Commit message: new swerve drive

File: urdf/2wv3(camera).urdf.xacro (robot description, xacro)
@@ -532,5 +532,5 @@
       <robot_param>robot_description</robot_param>
       <robot_param_node>robot_state_publisher</robot_param_node>
-      <parameters>/home/manfred/Projects/Vitrox/src/robot_urdf/config/diffdrive.yaml</parameters>
+      <parameters>$(find robot_urdf)/config/diffdrive.yaml</parameters>
     </plugin>
   </gazebo>

File: urdf/ranger1s_urdf_6.urdf.xacro (robot description, xacro)
@@ -13,15 +13,15 @@
     <inertial>
       <origin
-        xyz="-0.0031009 -4.9665E-19 -0.014767"
-        rpy="0 0 0" />
-      <mass
-        value="10" />
-      <inertia
-        ixx="4458"
-        ixy="-3.6838E-13"
-        ixz="-12.91"
-        iyy="5083.7"
-        iyz="-2.7411E-14"
-        izz="9008.3" />
+        xyz="-0.0057618 8.8769E-15 -0.033998"
+        rpy="0 0 0" />
+      <mass
+        value="32.713" />
+      <inertia
+        ixx="14.677"
+        ixy="-1.0477E-13"
+        ixz="-0.068414"
+        iyy="16.371"
+        iyz="-1.4749E-14"
+        izz="28.033" />
     </inertial>
     <visual>
@@ -36,5 +36,5 @@
         name="">
         <color
-          rgba="0.52941 0.54902 0.54902 1" />
+          rgba="0.89804 0.91765 0.92941 1" />
       </material>
     </visual>
@@ -71,46 +71,46 @@
   </joint>
   <link
-    name="wheel_holder_link">
-    <inertial>
-      <origin
-        xyz="1.1102E-16 0 -0.19944"
-        rpy="0 0 0" />
-      <mass
-        value="3" />
-      <inertia
-        ixx="4.7304"
-        ixy="-5.1035E-17"
-        ixz="-2.0355E-16"
-        iyy="4.794"
-        iyz="4.0941E-17"
-        izz="2.6221" />
-    </inertial>
-    <visual>
-      <origin
-        xyz="0 0 0"
-        rpy="0 0 0" />
-      <geometry>
-        <mesh
-          filename="package://robot_urdf/meshes/wheel_holder_link.STL" />
-      </geometry>
-      <material
-        name="">
-        <color
-          rgba="0.52941 0.54902 0.54902 1" />
-      </material>
-    </visual>
-    <collision>
-      <origin
-        xyz="0 0 0"
-        rpy="0 0 0" />
-      <geometry>
-        <mesh
-          filename="package://robot_urdf/meshes/wheel_holder_link.STL" />
-      </geometry>
-    </collision>
-  </link>
-  <joint
-    name="wheel_holder_joint"
-    type="fixed">
+    name="wheel_holder_link_lf">
+    <inertial>
+      <origin
+        xyz="1.1102E-16 -2.2204E-16 -0.2296"
+        rpy="0 0 0" />
+      <mass
+        value="4.2419" />
+      <inertia
+        ixx="0.1287"
+        ixy="-7.3591E-17"
+        ixz="-7.8137E-18"
+        iyy="0.13522"
+        iyz="1.4281E-16"
+        izz="0.079121" />
+    </inertial>
+    <visual>
+      <origin
+        xyz="0 0 0"
+        rpy="0 0 0" />
+      <geometry>
+        <mesh
+          filename="package://robot_urdf/meshes/wheel_holder_link_lf.STL" />
+      </geometry>
+      <material
+        name="">
+        <color
+          rgba="0.89804 0.91765 0.92941 1" />
+      </material>
+    </visual>
+    <collision>
+      <origin
+        xyz="0 0 0"
+        rpy="0 0 0" />
+      <geometry>
+        <mesh
+          filename="package://robot_urdf/meshes/wheel_holder_link_lf.STL" />
+      </geometry>
+    </collision>
+  </link>
+  <joint
+    name="wheel_holder_joint_lf"
+    type="revolute">
     <origin
       xyz="0.65801 0.7012 -0.42432"
@@ -119,8 +119,10 @@
       link="chassis_link" />
     <child
-      link="wheel_holder_link" />
+      link="wheel_holder_link_lf" />
     <axis
       xyz="0 0 1" />
     <limit
+      lower="0"
+      upper="0"
       effort="100"
       velocity="10" />
@@ -130,332 +132,5 @@
   </joint>
   <link
-    name="wheel_link">
-    <inertial>
-      <origin
-        xyz="0 1.1102E-16 -2.7756E-17"
-        rpy="0 0 0" />
-      <mass
-        value="1" />
-      <inertia
-        ixx="0.056856"
-        ixy="1.2844E-18"
-        ixz="6.163E-33"
-        iyy="0.11125"
-        iyz="9.1985E-31"
-        izz="0.056856" />
-    </inertial>
-    <visual>
-      <origin
-        xyz="0 0 0"
-        rpy="0 0 0" />
-      <geometry>
-        <mesh
-          filename="package://robot_urdf/meshes/wheel_link.STL" />
-      </geometry>
-      <material
-        name="">
-        <color
-          rgba="0.29804 0.29804 0.29804 1" />
-      </material>
-    </visual>
-    <collision>
-      <origin
-        xyz="0 0 0"
-        rpy="0 0 0" />
-      <geometry>
-        <mesh
-          filename="package://robot_urdf/meshes/wheel_link.STL" />
-      </geometry>
-    </collision>
-  </link>
-  <joint
-    name="wheel_joint"
-    type="continuous">
-    <origin
-      xyz="0 0 -0.35"
-      rpy="0 0 0" />
-    <parent
-      link="wheel_holder_link" />
-    <child
-      link="wheel_link" />
-    <axis
-      xyz="0 1 0" />
-    <limit
-      effort="10000"
-      velocity="10" />
-  </joint>
-  <link
-    name="wheel_holder_link_1">
-    <inertial>
-      <origin
-        xyz="1.1102E-16 0 -0.19944"
-        rpy="0 0 0" />
-      <mass
-        value="3" />
-      <inertia
-        ixx="4.7304"
-        ixy="5.1651E-17"
-        ixz="-2.7889E-16"
-        iyy="4.794"
-        iyz="1.2939E-16"
-        izz="2.6221" />
-    </inertial>
-    <visual>
-      <origin
-        xyz="0 0 0"
-        rpy="0 0 0" />
-      <geometry>
-        <mesh
-          filename="package://robot_urdf/meshes/wheel_holder_link_1.STL" />
-      </geometry>
-      <material
-        name="">
-        <color
-          rgba="0.52941 0.54902 0.54902 1" />
-      </material>
-    </visual>
-    <collision>
-      <origin
-        xyz="0 0 0"
-        rpy="0 0 0" />
-      <geometry>
-        <mesh
-          filename="package://robot_urdf/meshes/wheel_holder_link_1.STL" />
-      </geometry>
-    </collision>
-  </link>
-  <joint
-    name="wheel_holder_joint_1"
-    type="continuous">
-    <origin
-      xyz="-0.79256 0.7012 -0.42432"
-      rpy="0 0 0" />
-    <parent
-      link="chassis_link" />
-    <child
-      link="wheel_holder_link_1" />
-    <axis
-      xyz="0 0 1" />
-  </joint>
-  <link
-    name="wheel_link_1">
-    <inertial>
-      <origin
-        xyz="0 1.1102E-16 0"
-        rpy="0 0 0" />
-      <mass
-        value="1" />
-      <inertia
-        ixx="0.056856"
-        ixy="2.3141E-17"
-        ixz="-7.0617E-33"
-        iyy="0.11125"
-        iyz="1.0331E-31"
-        izz="0.056856" />
-    </inertial>
-    <visual>
-      <origin
-        xyz="0 0 0"
-        rpy="0 0 0" />
-      <geometry>
-        <mesh
-          filename="package://robot_urdf/meshes/wheel_link_1.STL" />
-      </geometry>
-      <material
-        name="">
-        <color
-          rgba="0.29804 0.29804 0.29804 1" />
-      </material>
-    </visual>
-    <collision>
-      <origin
-        xyz="0 0 0"
-        rpy="0 0 0" />
-      <geometry>
-        <mesh
-          filename="package://robot_urdf/meshes/wheel_link_1.STL" />
-      </geometry>
-    </collision>
-  </link>
-  <joint
-    name="wheel_joint_1"
-    type="continuous">
-    <origin
-      xyz="0 0 -0.35"
-      rpy="0 0 0" />
-    <parent
-      link="wheel_holder_link_1" />
-    <child
-      link="wheel_link_1" />
-    <axis
-      xyz="0 1 0" />
-    <limit
-      effort="10000"
-      velocity="10" />
-  </joint>
-  <link
-    name="wheel_holder_link_2">
-    <inertial>
-      <origin
-        xyz="0 0 -0.19944"
-        rpy="0 0 0" />
-      <mass
-        value="3" />
-      <inertia
-        ixx="4.7304"
-        ixy="-1.6561E-16"
-        ixz="2.4565E-16"
-        iyy="4.794"
-        iyz="-8.4193E-18"
-        izz="2.6221" />
-    </inertial>
-    <visual>
-      <origin
-        xyz="0 0 0"
-        rpy="0 0 0" />
-      <geometry>
-        <mesh
-          filename="package://robot_urdf/meshes/wheel_holder_link_2.STL" />
-      </geometry>
-      <material
-        name="">
-        <color
-          rgba="0.52941 0.54902 0.54902 1" />
-      </material>
-    </visual>
-    <collision>
-      <origin
-        xyz="0 0 0"
-        rpy="0 0 0" />
-      <geometry>
-        <mesh
-          filename="package://robot_urdf/meshes/wheel_holder_link_2.STL" />
-      </geometry>
-    </collision>
-  </link>
-  <joint
-    name="wheel_holder_joint_2"
-    type="continuous">
-    <origin
-      xyz="-0.79256 -0.7012 -0.42432"
-      rpy="0 0 0" />
-    <parent
-      link="chassis_link" />
-    <child
-      link="wheel_holder_link_2" />
-    <axis
-      xyz="0 0 1" />
-  </joint>
-  <link
-    name="wheel_link_2">
-    <inertial>
-      <origin
-        xyz="0 0 0"
-        rpy="0 0 0" />
-      <mass
-        value="1" />
-      <inertia
-        ixx="0.056856"
-        ixy="6.6322E-17"
-        ixz="-1.5426E-32"
-        iyy="0.11125"
-        iyz="-3.4376E-19"
-        izz="0.056856" />
-    </inertial>
-    <visual>
-      <origin
-        xyz="0 0 0"
-        rpy="0 0 0" />
-      <geometry>
-        <mesh
-          filename="package://robot_urdf/meshes/wheel_link_2.STL" />
-      </geometry>
-      <material
-        name="">
-        <color
-          rgba="0.29804 0.29804 0.29804 1" />
-      </material>
-    </visual>
-    <collision>
-      <origin
-        xyz="0 0 0"
-        rpy="0 0 0" />
-      <geometry>
-        <mesh
-          filename="package://robot_urdf/meshes/wheel_link_2.STL" />
-      </geometry>
-    </collision>
-  </link>
-  <joint
-    name="wheel_joint_2"
-    type="continuous">
-    <origin
-      xyz="0 0 -0.35"
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