Commit message: fixed urdf

File: urdf/ranger1s_urdf_6.urdf.xacro (robot description, xacro)
@@ -53,5 +53,5 @@
     type="fixed">
     <origin
-      xyz="0 0 0.96832"
+      xyz="0.067275 0 0.96832"
       rpy="0 0 0" />
     <parent
@@ -112,5 +112,5 @@
   <joint
     name="wheel_holder_joint_lf"
-    type="revolute">
+    type="continuous">
     <origin
       xyz="0.65801 0.7012 -0.42432"
@@ -122,12 +122,4 @@
     <axis
       xyz="0 0 1" />
-    <limit
-      lower="0"
-      upper="0"
-      effort="100"
-      velocity="10" />
-    <dynamics
-      damping="0.1"
-      friction="0.1" />
   </joint>
   <link
@@ -150,5 +142,5 @@
       <origin
         xyz="0 0 0"
-        rpy="0 0 0" />
+        rpy="1.570796 1.570796 0" />
       <geometry>
         <cylinder radius="0.194" length="0.05" />
@@ -163,5 +155,5 @@
       <origin
         xyz="0 0 0"
-        rpy="0 0 0" />
+        rpy="1.570796 1.570796 0" />
       <geometry>
         <cylinder radius="0.194" length="0.05" />
@@ -180,5 +172,5 @@
       link="wheel_link_lf" />
     <axis
-      xyz="0 -1 0" />
+      xyz="0 1 0" />
     <limit
       effort="100"
@@ -227,5 +219,5 @@
   <joint
     name="wheel_holder_joint_lb"
-    type="revolute">
+    type="continuous">
     <origin
       xyz="-0.79256 0.7012 -0.42432"
@@ -237,9 +229,4 @@
     <axis
       xyz="0 0 1" />
-    <limit
-      lower="0"
-      upper="0"
-      effort="100"
-      velocity="10" />
   </joint>
   <link
@@ -262,5 +249,5 @@
       <origin
         xyz="0 0 0"
-        rpy="0 0 0" />
+        rpy="1.570796 1.570796 0" />
       <geometry>
         <cylinder radius="0.194" length="0.05" />
@@ -275,5 +262,5 @@
       <origin
         xyz="0 0 0"
-        rpy="0 0 0" />
+        rpy="1.570796 1.570796 0" />
       <geometry>
         <cylinder radius="0.194" length="0.05" />
@@ -292,5 +279,5 @@
       link="wheel_link_lb" />
     <axis
-      xyz="0 -1 0" />
+      xyz="0 1 0" />
     <limit
       effort="100"
@@ -339,5 +326,5 @@
   <joint
     name="wheel_holder_joint_rb"
-    type="revolute">
+    type="continuous">
     <origin
       xyz="-0.79256 -0.7012 -0.42432"
@@ -349,9 +336,4 @@
     <axis
       xyz="0 0 1" />
-    <limit
-      lower="0"
-      upper="0"
-      effort="100"
-      velocity="10" />
   </joint>
   <link
@@ -374,5 +356,5 @@
       <origin
         xyz="0 0 0"
-        rpy="0 0 0" />
+        rpy="1.570796 1.570796 0" />
       <geometry>
         <cylinder radius="0.194" length="0.05" />
@@ -387,5 +369,5 @@
       <origin
         xyz="0 0 0"
-        rpy="0 0 0" />
+        rpy="1.570796 1.570796 0" />
       <geometry>
         <cylinder radius="0.194" length="0.05" />
@@ -404,5 +386,5 @@
       link="wheel_link_rb" />
     <axis
-      xyz="0 -1 0" />
+      xyz="0 1 0" />
     <limit
       effort="100"
@@ -451,5 +433,5 @@
   <joint
     name="wheel_holder_joint_rf"
-    type="revolute">
+    type="continuous">
     <origin
       xyz="0.65801 -0.7012 -0.42432"
@@ -461,9 +443,4 @@
     <axis
       xyz="0 0 1" />
-    <limit
-      lower="0"
-      upper="0"
-      effort="100"
-      velocity="10" />
   </joint>
   <link
@@ -486,5 +463,5 @@
       <origin
         xyz="0 0 0"
-        rpy="0 0 0" />
+        rpy="1.570796 1.570796 0" />
       <geometry>
         <cylinder radius="0.194" length="0.05" />
@@ -499,5 +476,5 @@
       <origin
         xyz="0 0 0"
-        rpy="0 0 0" />
+        rpy="1.570796 1.570796 0" />
       <geometry>
         <cylinder radius="0.194" length="0.05" />
@@ -516,5 +493,5 @@
       link="wheel_link_rf" />
     <axis
-      xyz="0 -1 0" />
+      xyz="0 1 0" />
     <limit
       effort="100"
@@ -522,16 +499,32 @@
   </joint>
   <link
-    name="depth_camera_link">
-  </link>
-  <joint
-    name="depth_camera_joint"
+    name="depth_link_r">
+  </link>
+  <joint
+    name="depth_joint_r"
     type="fixed">
     <origin
-      xyz="1.017 0 -0.21645"
-      rpy="0 0 0" />
+      xyz="1.017 -0.45 -0.21645"
+      rpy="0 0.7853982 0.2618" />
     <parent
       link="chassis_link" />
     <child
-      link="depth_camera_link" />
+      link="depth_link_r" />
+    <axis
+      xyz="0 0 0" />
+  </joint>
+  <link
+    name="depth_link_l">
+  </link>
+  <joint
+    name="depth_joint_l"
+    type="fixed">
+    <origin
+      xyz="1.017 0.45 -0.21645"
+      rpy="0 0.7853982 -0.2618" />
+    <parent
+      link="chassis_link" />
+    <child
+      link="depth_link_l" />
     <axis
       xyz="0 0 0" />
@@ -561,13 +554,44 @@
       <state_interface name="velocity" />
     </joint>
-    <!-- <joint name="wheel_holder_joint_1"> -->
-    <!--   <state_interface name="position" /> -->
-    <!--   <state_interface name="velocity" /> -->
-    <!-- </joint> -->
-    <!---->
-    <!-- <joint name="wheel_holder_joint_2"> -->
-    <!--   <state_interface name="position" /> -->
-    <!--   <state_interface name="velocity" /> -->
-    <!-- </joint> -->
+    <joint name="wheel_holder_joint_lf">
+      <state_interface name="position" />
+      <state_interface name="velocity" />
+      <command_interface name="position">
+        <param name="p">100.0</param>
+        <param name="i">0.05</param>
+        <param name="d">1.0</param>
+        <param name="max">100.0</param>
+      </command_interface>
+    </joint>
+    <joint name="wheel_holder_joint_rf">
+      <state_interface name="position" />
+      <state_interface name="velocity" />
+      <command_interface name="position">
+        <param name="p">100.0</param>
+        <param name="i">0.05</param>
+        <param name="d">1.0</param>
+        <param name="max">100.0</param>
+      </command_interface>
+    </joint>
+    <joint name="wheel_holder_joint_lb">
+      <state_interface name="position" />
+      <state_interface name="velocity" />
+      <command_interface name="position">
+        <param name="p">100.0</param>
+        <param name="i">0.05</param>
+        <param name="d">1.0</param>
+        <param name="max">100.0</param>
+      </command_interface>
+    </joint>
+    <joint name="wheel_holder_joint_rb">
+      <state_interface name="position" />
+      <state_interface name="velocity" />
+      <command_interface name="position">
+        <param name="p">100.0</param>
+        <param name="i">0.05</param>
+        <param name="d">1.0</param>
+        <param name="max">100.0</param>
+      </command_interface>
+    </joint>
   </ros2_control>
   <gazebo>
@@ -576,81 +600,109 @@
       <robot_param>robot_description</robot_param>
       <robot_param_node>robot_state_publisher</robot_param_node>
-      <parameters>$(find robot_urdf)/config/diffdrive_4w.yaml</parameters>
+      <parameters>$(find robot_urdf)/config/swerve_drive.yaml</parameters>
+      <!-- <ros>
+        <remapping>/ackermann_steering_controller/tf_odometry:=/tf</remapping>
+      </ros> -->
     </plugin>
   </gazebo>
   <gazebo reference="wheel_link_lf">
     <mu1>1.2</mu1>
-    <mu2>0.01</mu2>
+    <mu2>1.2</mu2>
     <kp>1000000.0</kp>
     <kd>100.0</kd>
+    <!-- <fdir1>1 0 0</fdir1> -->
   </gazebo>
   <gazebo reference="wheel_link_lb">
     <mu1>1.2</mu1>
-    <mu2>0.01</mu2>
+    <mu2>1.2</mu2>
     <kp>1000000.0</kp>
     <kd>100.0</kd>
+    <!-- <fdir1>1 0 0</fdir1> -->
   </gazebo>
   <gazebo reference="wheel_link_rb">
     <mu1>1.2</mu1>
-    <mu2>0.01</mu2>
+    <mu2>1.2</mu2>
     <kp>1000000.0</kp>
     <kd>100.0</kd>
+    <!-- <fdir1>1 0 0</fdir1> -->
   </gazebo>
   <gazebo reference="wheel_link_rf">
     <mu1>1.2</mu1>
-    <mu2>0.01</mu2>
+    <mu2>1.2</mu2>
     <kp>1000000.0</kp>
     <kd>100.0</kd>
+    <!-- <fdir1>1 0 0</fdir1> -->
   </gazebo>
   <gazebo reference="chassis_link">
     <material>Gazebo/Orange</material>
   </gazebo>
-  <gazebo reference="depth_camera_link">
-    <sensor name="rgbd_camera" type="rgbd_camera">
-      <ignition_frame_id>depth_camera_link</ignition_frame_id>
-      <camera name="rgbd_camera_frame">
-        <horizontal_fov>1.3962634</horizontal_fov>
-        <lens>
-          <intrinsics>
-            <fx>277.1</fx>
-            <fy>277.1</fy>
-            <cx>160.5</cx>
-            <cy>120.5</cy>
-            <s>0</s>
-          </intrinsics>
-        </lens>
-        <distortion>
-          <k1>0.104207</k1>
-          <k2>-0.255558</k2>
-          <k3>0.128694</k3>
-          <p1>0.000512</p1>
-          <p2>0.000319</p2>
-          <center>0.5 0.5</center>
-        </distortion>
-        <image>
-          <width>1280</width>
-          <height>720</height>
-          <format>L8</format>
-        </image>
-        <clip>
-          <near>0.01</near>
-          <far>300</far>
-        </clip>
-        <depth_camera>
-          <clip>
-            <near>0.1</near>
-            <far>10</far>
-          </clip>
-        </depth_camera>
+  <gazebo reference="depth_link_l">
+    <sensor name="depth_sensor_l" type="gpu_lidar">
+      <ignition_frame_id>depth_link_l</ignition_frame_id>
+      <topic>lidar_l</topic>
+      <update_rate>10</update_rate>
+      <always_on>true</always_on>
+      <visualize>false</visualize> <!-- Keep false to save resources unless debugging rays -->
+      <lidar>
+        <scan>
+          <horizontal>
+            <samples>360</samples>
+            <resolution>1</resolution>
+            <min_angle>-0.50705</min_angle>
+            <max_angle>0.50705</max_angle>
+          </horizontal>
+          <vertical>
+            <samples>100</samples> <!-- 16 vertical slices provides a good 3D point cloud -->
+            <resolution>1</resolution>
+            <min_angle>-0.39445</min_angle> <!-- -15 degrees -->
+            <max_angle>0.39445</max_angle>  <!-- +15 degrees -->
+          </vertical>
+        </scan>
+        <range>
+          <min>0.1</min>
+          <max>15.0</max> <!-- 15 meter range is typical -->
+          <resolution>0.01</resolution>
+        </range>
         <noise>
           <type>gaussian</type>
-          <mean>0</mean>
-          <stddev>0.003</stddev>
+          <mean>0.0</mean>
+          <stddev>0.01</stddev>
         </noise>
-      </camera>
-      <always_on>1</always_on>
+      </lidar>
+    </sensor>
+  </gazebo>
+  <gazebo reference="depth_link_r">
+    <sensor name="depth_sensor_r" type="gpu_lidar">
+      <ignition_frame_id>depth_link_r</ignition_frame_id>
+      <topic>lidar_r</topic>
       <update_rate>10</update_rate>
-      <visualize>0</visualize>
-      <topic>depth_camera</topic>
+      <always_on>true</always_on>
+      <visualize>false</visualize>
+      <lidar>
+        <scan>
+          <horizontal>
+            <samples>360</samples>
+            <resolution>1</resolution>
+            <min_angle>-0.50705</min_angle>
+            <max_angle>0.50705</max_angle>
+          </horizontal>
+          <vertical>
+            <samples>100</samples>
+            <resolution>1</resolution>
+            <min_angle>-0.39445</min_angle>
+            <max_angle>0.39445</max_angle>
+          </vertical>
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